File: adadad/adadad.kicad_pcb (KiCad board)
At the start: 2 copper layers, 31 x 99.5 mm, 34 parts, among them J1 Conn_02x05_Odd_Even, Q1 BC547, Q2 BC547, Q3 BC547, U1 ICM7555, U2 TL074

Commit message: All kinds of stuff
Parts:
- added U3: TL074, Package_DIP:DIP-14_W7.62mm_Socket, F.Cu at (122.5, 108.5)
- U2: footprint Package_DIP:DIP-14_W10.16mm -> Package_DIP:DIP-14_W7.62mm_Socket
- moved D1 42.2 mm to (130.5, 63.0), turned to 90 degrees
- moved RV2 28.3 mm to (113.5, 91.0), turned to 180 degrees
- moved D7 19.9 mm to (119.0, 115.0), turned to 180 degrees
- moved RV1 16.0 mm to (129.5, 103.5)
- moved C4 12.5 mm to (106.5, 93.5)
- moved G*** 8.32 mm to (118.0, 98.0)
- moved J1 4.27 mm to (125.5, 84.5)
- moved Q1 2.55 mm to (122.5, 61.0)
- moved Q2 2.55 mm to (122.5, 51.0)
- moved Q3 2.55 mm to (122.5, 56.0)
- moved C2 2.06 mm to (123.0, 66.0)
- moved U1 2.06 mm to (130.5, 77.0)
- moved U2 1.12 mm to (130.0, 143.5)
Connections:
- GATE_J2 pad T: Net-(D1-Pad1) -> Net-(GATE_J2-PadT)
- R10 pad 2: Net-(C3-Pad2) -> Net-(R10-Pad2)
- RV2 pad 1: Net-(C3-Pad2) -> Net-(RV2-Pad1)
- U2 pad 1: Net-(OUT_J4-PadT) -> Net-(U2-Pad1)
- U2 pad 10: GND -> (no net)
- U2 pad 12: (no net) -> Net-(GATE_J2-PadT)
- U2 pad 13: (no net) -> Net-(D1-Pad1)
- U2 pad 14: (no net) -> Net-(D1-Pad1)
- U2 pad 2: Net-(OUT_J4-PadT) -> Net-(U2-Pad1)
- U2 pad 5: Net-(RV1-Pad2) -> Net-(U2-Pad1)
- U2 pad 6: Net-(RV2-Pad2) -> Net-(OUT_J4-PadT)
- U2 pad 7: Net-(D6-Pad2) -> Net-(OUT_J4-PadT)
- U2 pad 8: Net-(D4-Pad1) -> (no net)
- U2 pad 9: Net-(D4-Pad2) -> (no net)
Routing:
- net Net-(GATE_J2-PadT): track 0.00 -> 46.0 mm
- net Net-(D1-Pad1): track 60.2 -> 101.3 mm
- net Net-(RV2-Pad1): track 0.00 -> 36.5 mm
- net Net-(U2-Pad1): track 0.00 -> 36.1 mm
- net Net-(C3-Pad2): track 131.3 -> 105.9 mm
- net Net-(R10-Pad2): track 0.00 -> 25.2 mm
- net -12V: track 69.2 -> 92.0 mm, vias 0 -> 1
- net Net-(D4-Pad2): track 45.5 -> 33.7 mm
- net Net-(Q2-Pad2): track 31.7 -> 20.2 mm
- net Net-(D6-Pad2): track 40.4 -> 51.6 mm, vias 0 -> 1
- net Net-(OUT_J4-PadT): track 39.5 -> 28.9 mm
- net Net-(Q3-Pad1): track 45.6 -> 36.9 mm
- net Net-(D4-Pad1): track 30.3 -> 37.5 mm
- net Net-(RV1-Pad2): track 15.8 -> 11.9 mm
- net Net-(C1-Pad2): track 55.4 -> 51.6 mm, vias 1 -> 0
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Other:
- board size 31 x 99.5 mm -> 30.5 x 99.5 mm
