File: adadad/adadad.sch (KiCad schematic (older format))
At the start: 33 parts, among them J1 Conn_02x05_Odd_Even, Q1 BC547, Q2 BC547, Q3 BC547, U1 ICM7555, U2 TL074

Commit message: All kinds of stuff
Parts:
- added unit 4 of U2
- added unit 1 of U3
- added unit 5 of U3
- added unit 3 of U3
- added unit 2 of U3
- EoC_J1, GATE_J2, OUT_J4: symbol Connector:AudioJack3_Ground -> audiojack2_ground_switch_numeric:AudioJack3_Ground
- U2: footprint Package_DIP:DIP-14_W10.16mm -> Package_DIP:DIP-14_W7.62mm_Socket
- renumbered U2 to U3
Connections:
- wire segments 121 -> 149
Other:
- moved on the sheet: D4, D6, D7, R10, RV1, RV2, U2B
