File: plastik/hardware/plastik.kicad_pcb (KiCad board)
At the start: 2 copper layers, 98 x 99.5 mm, 38 parts, among them J1 CV1, J10 AudioJack2_Ground_Switch, J11 AudioJack2_Ground_Switch, J2 CV2, J3 CV3, J4 CV4, J5 AudioJack2_Ground_Switch, J6 AudioJack2_Ground_Switch, J7 AudioJack2_Ground_Switch, J8 AudioJack2_Ground_Switch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

Commit message: All kinds of stuff
Parts:
- added G***: LOGO, fox_small, B.Cu at (137.0, 48.0)
